File: Schematics/Remote.sch (KiCad schematic (older format))
At the start: 9 parts

Commit message: schematic and  PCB Layout done..
Parts:
- removed IC?: ATTINY85-P, DIP8, symbol ATTINY85-P
- removed Q?: BC817-40, SOT-23, symbol BC817-40
- added IC1: meinTiny85, Sockets_DIP:DIP-8__300, symbol meinTiny85
- added P1, P2: CONN_01X01, Connect:1pin, symbol CONN_01X01
- added Q1: Q_NPN_CBE, Housings_TO-92:TO-92_Inline_Wide, symbol Q_NPN_CBE
- D1, D2: renamed from D?; footprint (none) -> LEDs:LED-5MM
- R1: renamed from R?; value R -> 1k; footprint (none) -> Resistors_ThroughHole:Resistor_Horizontal_RM10mm
- R2: renamed from R?; value R -> 150; footprint (none) -> Resistors_ThroughHole:Resistor_Horizontal_RM10mm
- SW1, SW2, SW3: renamed from SW?; footprint (none) -> meins:JTP-1130
Connections:
- net labels added: +BATT, GND
- wire segments 0 -> 26
- no-connect marks 0 -> 1
Other:
- note added: "Release"
- note added: "Reset"
- note added: "Timer"
- moved on the sheet: D1, D2, R1, R2, SW1, SW2, SW3
